File: BMS KiCad/BMS_v1.0/BMS_v1.0.kicad_sch (KiCad schematic)
At the start: 14 parts, among them J3 Conn_01x06, SW1 SW_Push, U1 STM32F103C6Tx, Y1 Resonator

Commit message: cell taps and passive balancing and cell to cell capacitors completed
Other:
- added sheet Battery Monitoring (Battery_Monitoring.kicad_sch)
Changed lines of the file:
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@@
+		)
+	)
+	(sheet
+		(at 194.056 98.806)
+		(size 22.352 9.906)
+		(exclude_from_sim no)
+		(in_bom yes)
+		(on_board yes)
+		(dnp no)
+		(fields_autoplaced yes)
+		(stroke
+			(width 0.1524)
+			(type solid)
+		)
+		(fill
+			(color 0 0 0 0.0000)
+		)
+		(property "Sheetname" "Battery Monitoring"
+			(at 194.056 98.0944 0)
+			(effects
+				(font
+					(size 1.27 1.27)
+				)
+				(justify left bottom)
+			)
+		)
+		(property "Sheetfile" "Battery_Monitoring.kicad_sch"
+			(at 194.056 109.2966 0)
+			(effects
+				(font
+					(size 1.27 1.27)
+				)
+				(justify left top)
+			)
+		)
+		(instances
+			(project "BMS_v1.0"
+				(path "/2822dab8-353f-4caa-aeee-4463efcfd06e"
+					(page "3")
+				)
+			)
 		)
 	)

Commit message: TI IC done except for I2C and precharge circuit
Other:
- note added: "find io pin for this"
Changed lines of the file:
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@@
+		)
+	)
+	(text "find io pin for this \n"
+		(exclude_from_sim no)
+		(at 163.576 75.692 0)
+		(effects
+			(font
+				(size 1.27 1.27)
+			)
 		)
 	)
@@
 		)
 	)
+	(global_label "DFETOFF"
+		(shape input)
+		(at 158.75 69.85 0)
+		(fields_autoplaced yes)
+		(effects
+			(font
+				(size 1.27 1.27)
+			)
+			(justify left)
+		)
+		(property "Intersheetrefs" "${INTERSHEET_REFS}"
+			(at 169.7181 69.85 0)
+			(effects
+				(font
+					(size 1.27 1.27)
+				)
+				(justify left)
+				(hide yes)
+			)
+		)
+	)
 	(global_label "NRST"
 		(shape input)
@@
 		)
 	)
+	(global_label "RST_SHUT"
+		(shape input)
+		(at 158.75 67.31 0)
+		(fields_autoplaced yes)
+		(effects
+			(font
+				(size 1.27 1.27)
+			)
+			(justify left)
+		)
+		(property "Intersheetrefs" "${INTERSHEET_REFS}"
+			(at 170.988 67.31 0)
+			(effects
+				(font
+					(size 1.27 1.27)
+				)
+				(justify left)
+				(hide yes)
+			)
+		)
+	)
 	(global_label "SWDIO"
 		(shape input)
@@
 		)
 	)
+	(global_label "CFETOFF"
+		(shape input)
+		(at 158.75 72.39 0)
+		(fields_autoplaced yes)
+		(effects
+			(font
+				(size 1.27 1.27)
+			)
+			(justify left)
+		)
+		(property "Intersheetrefs" "${INTERSHEET_REFS}"
+			(at 169.7181 72.39 0)
+			(effects
+				(font
+					(size 1.27 1.27)
+				)
+				(justify left)
+				(hide yes)
+			)
+		)
+	)
 	(symbol
 		(lib_id "Connector_Generic:Conn_01x06")
@@
 	)
 	(sheet
-		(at 54.102 42.418)
-		(size 14.478 6.35)
+		(at 164.592 47.244)
+		(size 19.812 9.652)
 		(exclude_from_sim no)
 		(in_bom yes)
@@
 		)
 		(property "Sheetname" "Power Protection"
-			(at 54.102 41.7064 0)
+			(at 164.592 46.5324 0)
 			(effects
 				(font
@@
 		)
 		(property "Sheetfile" "Power Protection.kicad_sch"
-			(at 54.102 49.3526 0)
+			(at 164.592 57.4806 0)
 			(effects
 				(font
@@
 	)
 	(sheet
-		(at 194.056 98.806)
+		(at 200.406 46.99)
 		(size 22.352 9.906)
 		(exclude_from_sim no)
@@
 		)
 		(property "Sheetname" "Battery Monitoring"
-			(at 194.056 98.0944 0)
+			(at 200.406 46.2784 0)
 			(effects
 				(font
@@
 		)
 		(property "Sheetfile" "Battery_Monitoring.kicad_sch"
-			(at 194.056 109.2966 0)
-			(effects
-				(font
+			(at 200.406 57.4806 0)
+			(effects
+				(font

Commit message: footprints for almost everything
Parts:
- C1, C2, C3, C4, C5, C6, C7, C8, C9: footprint (none) -> Capacitor_SMD:C_0603_1608Metric_Pad1.08x0.95mm_HandSolder
- R1: footprint (none) -> Fuse:Fuse_0603_1608Metric_Pad1.05x0.95mm_HandSolder
Changed lines of the file:
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@@
 			)
 		)
-		(property "Footprint" ""
+		(property "Footprint" "Capacitor_SMD:C_0603_1608Metric_Pad1.08x0.95mm_HandSolder"
 			(at 143.2052 31.496 0)
 			(effects
@@
 			)
 		)
-		(property "Footprint" ""
+		(property "Footprint" "Capacitor_SMD:C_0603_1608Metric_Pad1.08x0.95mm_HandSolder"
 			(at 113.4872 31.496 0)
 			(effects
@@
 			)
 		)
-		(property "Footprint" ""
+		(property "Footprint" "Capacitor_SMD:C_0603_1608Metric_Pad1.08x0.95mm_HandSolder"
 			(at 103.5812 31.496 0)
 			(effects
@@
 			)
 		)
-		(property "Footprint" ""
+		(property "Footprint" "Fuse:Fuse_0603_1608Metric_Pad1.05x0.95mm_HandSolder"
 			(at 101.092 76.454 90)
 			(effects
@@
 			)
 		)
-		(property "Footprint" ""
+		(property "Footprint" "Capacitor_SMD:C_0603_1608Metric_Pad1.08x0.95mm_HandSolder"
 			(at 167.3352 31.496 0)
 			(effects
@@
 			)
 		)
-		(property "Footprint" ""
+		(property "Footprint" "Capacitor_SMD:C_0603_1608Metric_Pad1.08x0.95mm_HandSolder"
 			(at 175.9712 31.496 0)
 			(effects
@@
 			)
 		)
-		(property "Footprint" ""
+		(property "Footprint" "Capacitor_SMD:C_0603_1608Metric_Pad1.08x0.95mm_HandSolder"
 			(at 133.2992 31.496 0)
 			(effects
@@
 			)
 		)
-		(property "Footprint" ""
+		(property "Footprint" "Capacitor_SMD:C_0603_1608Metric_Pad1.08x0.95mm_HandSolder"
 			(at 152.6032 31.496 0)
 			(effects
@@
 			)
 		)
-		(property "Footprint" ""
+		(property "Footprint" "Capacitor_SMD:C_0603_1608Metric_Pad1.08x0.95mm_HandSolder"
 			(at 90.3732 73.152 0)
 			(effects
@@
 			)
 		)
-		(property "Footprint" ""
+		(property "Footprint" "Capacitor_SMD:C_0603_1608Metric_Pad1.08x0.95mm_HandSolder"
 			(at 123.3932 31.496 0)
 			(effects
